Commit message: Usa parámetros compartidos de meshes en xacro

File: puzzlebot_description/urdf/base/puzzlebot_base.urdf.xacro (robot description, xacro)
@@ -12,5 +12,5 @@
       <origin xyz="0.0 0.0 0.0" rpy="0.0 0.0 0.0"/>
       <geometry>
-        <mesh filename="file://$(find puzzlebot_description)/meshes/Robot_lidar_base/Puzzlebot_Jetson_Lidar_Edition_Base.stl" scale="1 1 1"/>
+        <mesh filename="${mesh_puzzlebot_chassis}" scale="1 1 1"/>
       </geometry>
       <material name="white">
@@ -34,5 +34,5 @@
       <origin xyz="0.0 0.0 0.0" rpy="1.5708 0.0 0.0"/>
       <geometry>
-        <mesh filename="file://$(find puzzlebot_description)/meshes/Wheels/Puzzlebot_Wheel.stl" scale="1 1 1"/>
+        <mesh filename="${mesh_puzzlebot_wheel}" scale="1 1 1"/>
       </geometry>
       <material name="black">
@@ -56,5 +56,5 @@
       <origin xyz="0.0 0.0 0.0" rpy="1.5708 0.0 0.0"/>
       <geometry>
-        <mesh filename="file://$(find puzzlebot_description)/meshes/Wheels/Puzzlebot_Wheel.stl" scale="1 1 1"/>
+        <mesh filename="${mesh_puzzlebot_wheel}" scale="1 1 1"/>
       </geometry>
       <material name="black">
@@ -78,5 +78,5 @@
       <origin xyz="0.0 0.0 0.0" rpy="0.0 0.0 0.0"/>
       <geometry>
-        <mesh filename="file://$(find puzzlebot_description)/meshes/Components/Puzzlebot_Caster_Wheel.stl" scale="1 1 1"/>
+        <mesh filename="${mesh_puzzlebot_caster}" scale="1 1 1"/>
       </geometry>
       <material name="black">

File: puzzlebot_description/urdf/puzzlebot.xacro (robot description, xacro)
@@ -3,4 +3,5 @@
 <robot name="puzzlebot" xmlns:xacro="http://www.ros.org/wiki/xacro">
   <xacro:arg name="prefix" default="" />
+  <xacro:include filename="$(find puzzlebot_description)/urdf/sensors/parameters_jetson_lidar_ed.xacro"/>
   <xacro:include filename="$(find puzzlebot_description)/urdf/base/puzzlebot_base.urdf.xacro"/>
   <xacro:include filename="$(find puzzlebot_description)/urdf/sensors/macros.xacro"/>
@@ -8,4 +9,6 @@
   <xacro:puzzlebot_control prefix="$(arg prefix)"/> <!-- macro -->
   <xacro:include filename="$(find puzzlebot_description)/urdf/sensors/lidar.xacro"/>
-  <xacro:rpi_lidar_sensor prefix="$(arg prefix)"/> <!-- macro -->
+  <xacro:rpi_lidar_sensor
+    prefix="$(arg prefix)"
+    mesh_file="${mesh_puzzlebot_lidar}"/> <!-- macro -->
 </robot>

File: puzzlebot_description/urdf/sensors/parameters_jetson_lidar_ed.xacro (robot description, xacro)
@@ -165,7 +165,7 @@
             <xacro:property name="jetson_pos_w" value="0.0"/>
     <!--Meshes -->
-        <xacro:property name="mesh_puzzlebot_chassis"  value="$(find puzzlebot_description)/meshes/bases/Puzzlebot_Jetson_Lidar_Edition_Base.stl" />
-        <xacro:property name="mesh_puzzlebot_wheel"  value="$(find puzzlebot_description)/meshes/wheels/Puzzlebot_Wheel.stl" />
-        <xacro:property name="mesh_puzzlebot_caster"  value="$(find puzzlebot_description)/meshes/wheels/Puzzlebot_Caster_Wheel.stl" />
-        <xacro:property name="mesh_puzzlebot_jetson"  value="$(find puzzlebot_description)/meshes/misc/NVIDIA_Jetson.stl" />
+        <xacro:property name="mesh_puzzlebot_chassis"  value="file://$(find puzzlebot_description)/meshes/Robot_lidar_base/Puzzlebot_Jetson_Lidar_Edition_Base.stl" />
+        <xacro:property name="mesh_puzzlebot_wheel"  value="file://$(find puzzlebot_description)/meshes/Wheels/Puzzlebot_Wheel.stl" />
+        <xacro:property name="mesh_puzzlebot_caster"  value="file://$(find puzzlebot_description)/meshes/Components/Puzzlebot_Caster_Wheel.stl" />
+        <xacro:property name="mesh_puzzlebot_lidar"  value="file://$(find puzzlebot_description)/meshes/Sensor/RPLidar.stl" />
 </robot>
