Commit message: lidar adjustments

File: puzzlebot_description/urdf/sensors/lidar.xacro (robot description, xacro)
@@ -6,5 +6,5 @@
     frame_name:='laser_frame'
     parent:='base_link'
-    mesh_file:='file://$(find puzzlebot_description)/meshes/Sensor/RPLidar.stl'
+    mesh_file:='package://puzzlebot_description/meshes/Sensor/RPLidar.stl'
     lidar_base_mass:='0.1755'
     lidar_base_length:='0.08'

File: puzzlebot_description/urdf/sensors/parameters_jetson_lidar_ed.xacro (robot description, xacro)
@@ -165,7 +165,7 @@
             <xacro:property name="jetson_pos_w" value="0.0"/>
     <!--Meshes -->
-        <xacro:property name="mesh_puzzlebot_chassis"  value="file://$(find puzzlebot_description)/meshes/Robot_lidar_base/Puzzlebot_Jetson_Lidar_Edition_Base.stl" />
-        <xacro:property name="mesh_puzzlebot_wheel"  value="file://$(find puzzlebot_description)/meshes/Wheels/Puzzlebot_Wheel.stl" />
-        <xacro:property name="mesh_puzzlebot_caster"  value="file://$(find puzzlebot_description)/meshes/Components/Puzzlebot_Caster_Wheel.stl" />
-        <xacro:property name="mesh_puzzlebot_lidar"  value="file://$(find puzzlebot_description)/meshes/Sensor/RPLidar.stl" />
+        <xacro:property name="mesh_puzzlebot_chassis"  value="package://puzzlebot_description/meshes/Robot_lidar_base/Puzzlebot_Jetson_Lidar_Edition_Base.stl" />
+        <xacro:property name="mesh_puzzlebot_wheel"  value="package://puzzlebot_description/meshes/Wheels/Puzzlebot_Wheel.stl" />
+        <xacro:property name="mesh_puzzlebot_caster"  value="package://puzzlebot_description/meshes/Components/Puzzlebot_Caster_Wheel.stl" />
+        <xacro:property name="mesh_puzzlebot_lidar"  value="package://puzzlebot_description/meshes/Sensor/RPLidar.stl" />
 </robot>
